File: pcb-040/Matrix.kicad_sch (KiCad schematic)
At the start: 145 parts

Commit message: Update readme and add firmware
Parts:
- added MX15.125, MX27.15, MX81.15, MX93.125: MX-NoLED, MX_Only:MXOnly-1U-NoLED, symbol MX_Alps_Hybrid:MX-NoLED
Connections:
- net COL0: now also MX15.125.1 (COL)
- net COL1: now also MX27.15.1 (COL)
- net COL5: now also MX81.15.1 (COL)
- net COL6: now also MX93.125.1 (COL)
- net at D81.2 (A), MX81.2 (ROW): now also MX81.15.2 (ROW)
- net at D93.2 (A), MX93.2 (ROW): now also MX93.125.2 (ROW)
- net at D15.2 (A), MX15.2 (ROW): now also MX15.125.2 (ROW)
- net at D27.2 (A), MX27.2 (ROW): now also MX27.15.2 (ROW)
